File: 5uH_LISN.kicad_sch (KiCad schematic)
At the start: 75 parts, among them J1 Conn_SMA, J2 Conn_SMA, J3 BANANA_CONN, J4 BANANA_CONN, J5 BANANA_CONN, J6 BANANA_CONN, J7 BANANA_CONN, J8 BANANA_CONN

Commit message: redesign, see readme
Parts:
- removed CASE_HAMMOND_1590BBK1: ~, symbol CASE_HAMMOND_1590BBK:CASE_HAMMOND_1590BBK
- removed GD1, GD2: S30-A75X, 5uH_LISN:S30-A400X, symbol 5uH_LISN-eagle-import:GDT_2pin_correct
- removed J3, J4, J5, J6, J7, J8: BANANA_CONN, 5uH_LISN:BANANA_CONN, symbol 5uH_LISN-eagle-import:BANANA_CONN
- removed L12, L6: 1mH, 5uH_LISN:COILCRAFT_1008PS, symbol 5uH_LISN-eagle-import:INDUCTOR
- added CASE1: B013BK, 5uH_LISN:B013BK, symbol Gainta:B013BK
- added FID1, FID2, FID3: Fiducial, Fiducial:Fiducial_1mm_Mask2mm, symbol Mechanical:Fiducial
- added J3, J4, J5, J6, J7, J8: BANANA_CONN, 5uH_LISN:6,1-PAD, symbol 5uH_LISN:BANANA_CONN
- added L7, L8: 1mH, Inductor_SMD:L_1210_3225Metric, symbol Device:L
- added RF1: 132360, 5uH_LISN:RF_CAP, symbol 5uH_LISN:RF
- added U1, U2: SMD75XM, Fuse:Fuse_1812_4532Metric, symbol 5uH_LISN:SMD75XM
- C1, C2: symbol 5uH_LISN-rescue:C-Device -> Device:C; Manufacturer TDK -> (none); Part number (none) -> KRM55WR72A226MH01L; manf# CKG57NX7S2A226M500JH -> (none)
- C10: renamed from C14; symbol 5uH_LISN-eagle-import:C-EUC0805 -> Device:C; Manufacturer AVX -> (none); Part number (none) -> CC0805KKX7R0BB474; manf# 08051C474KAT2A -> (none)
- C11: renamed from C15; symbol 5uH_LISN-eagle-import:C-EUC1206 -> Device:C; Manufacturer TDK -> (none); Part number (none) -> CC1206KKX7RYBB104; manf# C3216X7R2E104K160AA -> (none)
- C12: renamed from C16; symbol 5uH_LISN-eagle-import:C-EUC1206 -> Device:C; Manufacturer TDK -> (none); Part number (none) -> CC1206KKX7RYBB104; manf# C3216X7R2E104K160AA -> (none)
- C3: renamed from C5; symbol 5uH_LISN-rescue:C-Device -> Device:C; Manufacturer TDK -> (none); Part number (none) -> CC1210KKX7R0BB225; manf# CGA6N3X7R2A225K230AB -> (none)
- C4: renamed from C6; symbol 5uH_LISN-rescue:C-Device -> Device:C; Manufacturer TDK -> (none); Part number (none) -> CC1210KKX7R0BB225; manf# CGA6N3X7R2A225K230AB -> (none)
- C5: renamed from C7; symbol 5uH_LISN-rescue:C-Device -> Device:C; Manufacturer TDK -> (none); Part number (none) -> CC1210KKX7R0BB225; manf# CGA6N3X7R2A225K230AB -> (none)
- C6: renamed from C8; symbol 5uH_LISN-rescue:C-Device -> Device:C; Manufacturer TDK -> (none); Part number (none) -> CC1210KKX7R0BB225; manf# CGA6N3X7R2A225K230AB -> (none)
- C7: renamed from C11; symbol 5uH_LISN-eagle-import:C-EUC0805 -> Device:C; Manufacturer AVX -> (none); Part number (none) -> CC0805KKX7R0BB474; manf# 08051C474KAT2A -> (none)
- C8: renamed from C12; symbol 5uH_LISN-eagle-import:C-EUC0805 -> Device:C; Manufacturer AVX -> (none); Part number (none) -> CC0805KKX7R0BB474; manf# 08051C474KAT2A -> (none)
- C9: renamed from C13; symbol 5uH_LISN-eagle-import:C-EUC0805 -> Device:C; Manufacturer AVX -> (none); Part number (none) -> CC0805KKX7R0BB474; manf# 08051C474KAT2A -> (none)
- D1: renamed from D3; value SOT23-DIODEDUAL -> BAV99,215; symbol SOT23-DIODEDUAL:SOT23-DIODEDUAL -> Device:D_Dual_Series_AKC_Parallel; LCSC C2500 -> (none); Manufacturer Nexperia -> (none); Part number (none) -> BAV99,215; manf# BAV99,215 -> (none)
- D2: renamed from D1; value SOT23-DIODEDUAL -> BAV99,215; symbol SOT23-DIODEDUAL:SOT23-DIODEDUAL -> Device:D_Dual_Series_AKC_Parallel; LCSC C2500 -> (none); Manufacturer Nexperia -> (none); Part number (none) -> BAV99,215; manf# BAV99,215 -> (none)
- D3: renamed from D2; value SOT23-DIODEDUAL -> BAV99,215; symbol SOT23-DIODEDUAL:SOT23-DIODEDUAL -> Device:D_Dual_Series_AKC_Parallel; LCSC C2500 -> (none); Manufacturer Nexperia -> (none); Part number (none) -> BAV99,215; manf# BAV99,215 -> (none)
- D4: value SOT23-DIODEDUAL -> BAV99,215; symbol SOT23-DIODEDUAL:SOT23-DIODEDUAL -> Device:D_Dual_Series_AKC_Parallel; LCSC C2500 -> (none); Manufacturer Nexperia -> (none); Part number (none) -> BAV99,215; manf# BAV99,215 -> (none)
- H1, H2, H3, H4: now not fitted; now left out of the parts list
- J1, J2: footprint Connector_Coaxial:SMA_Wurth_60312002114503_Vertical -> Connector_Coaxial:SMB_Jack_Vertical; Manufacturer TE -> (none); Part number (none) -> KLS1-SMA001; manf# 5-1814832-2 -> (none)
- L1: renamed from L7; value 1.1uH -> 1.0uH; footprint 5uH_LISN:WE-HCI_7030_7040_7050 -> 5uH_LISN:SMS1040; symbol 5uH_LISN-eagle-import:WE-HCI_7030_7040_7050 -> Device:L; Manufacturer Wurth / Würth -> (none); Part number (none) -> SMS1040-1R0MT; manf# 744314110 -> (none)
- L10: value 1.1uH -> 1.0uH; footprint 5uH_LISN:WE-HCI_7030_7040_7050 -> 5uH_LISN:SMS1040; symbol 5uH_LISN-eagle-import:WE-HCI_7030_7040_7050 -> Device:L; Manufacturer Wurth / Würth -> (none); Part number (none) -> SMS1040-1R0MT; manf# 744314110 -> (none)
- L11: renamed from L5; value 1.1uH -> 1.0uH; footprint 5uH_LISN:WE-HCI_7030_7040_7050 -> 5uH_LISN:SMS1040; symbol 5uH_LISN-eagle-import:WE-HCI_7030_7040_7050 -> Device:L; Manufacturer Wurth / Würth -> (none); Part number (none) -> SMS1040-1R0MT; manf# 744314110 -> (none)
- L12: renamed from L11; value 1.1uH -> 1.0uH; footprint 5uH_LISN:WE-HCI_7030_7040_7050 -> 5uH_LISN:SMS1040; symbol 5uH_LISN-eagle-import:WE-HCI_7030_7040_7050 -> Device:L; Manufacturer Wurth / Würth -> (none); Part number (none) -> SMS1040-1R0MT; manf# 744314110 -> (none)
- L2: renamed from L1; value 1.1uH -> 1.0uH; footprint 5uH_LISN:WE-HCI_7030_7040_7050 -> 5uH_LISN:SMS1040; symbol 5uH_LISN-eagle-import:WE-HCI_7030_7040_7050 -> Device:L; Manufacturer Wurth / Würth -> (none); Part number (none) -> SMS1040-1R0MT; manf# 744314110 -> (none)
- L3: renamed from L2; value 1.1uH -> 1.0uH; footprint 5uH_LISN:WE-HCI_7030_7040_7050 -> 5uH_LISN:SMS1040; symbol 5uH_LISN-eagle-import:WE-HCI_7030_7040_7050 -> Device:L; Manufacturer Wurth / Würth -> (none); Part number (none) -> SMS1040-1R0MT; manf# 744314110 -> (none)
- L4: renamed from L8; value 1.1uH -> 1.0uH; footprint 5uH_LISN:WE-HCI_7030_7040_7050 -> 5uH_LISN:SMS1040; symbol 5uH_LISN-eagle-import:WE-HCI_7030_7040_7050 -> Device:L; Manufacturer Wurth / Würth -> (none); Part number (none) -> SMS1040-1R0MT; manf# 744314110 -> (none)
- L5: renamed from L3; value 1.1uH -> 1.0uH; footprint 5uH_LISN:WE-HCI_7030_7040_7050 -> 5uH_LISN:SMS1040; symbol 5uH_LISN-eagle-import:WE-HCI_7030_7040_7050 -> Device:L; Manufacturer Wurth / Würth -> (none); Part number (none) -> SMS1040-1R0MT; manf# 744314110 -> (none)
- L6: renamed from L9; value 1.1uH -> 1.0uH; footprint 5uH_LISN:WE-HCI_7030_7040_7050 -> 5uH_LISN:SMS1040; symbol 5uH_LISN-eagle-import:WE-HCI_7030_7040_7050 -> Device:L; Manufacturer Wurth / Würth -> (none); Part number (none) -> SMS1040-1R0MT; manf# 744314110 -> (none)
- L9: renamed from L4; value 1.1uH -> 1.0uH; footprint 5uH_LISN:WE-HCI_7030_7040_7050 -> 5uH_LISN:SMS1040; symbol 5uH_LISN-eagle-import:WE-HCI_7030_7040_7050 -> Device:L; Manufacturer Wurth / Würth -> (none); Part number (none) -> SMS1040-1R0MT; manf# 744314110 -> (none)
- R1, R2: symbol 5uH_LISN-eagle-import:R-EU_R0805 -> Device:R; Manufacturer TE -> (none); Part number (none) -> PTFR0805B909RP9; manf# RQ73C2A909RBTD -> (none)
- R10, R13, R14, R9: symbol 5uH_LISN-rescue:R-Device -> Device:R; Manufacturer YAGEO -> (none); Part number (none) -> RC1206JR-7W0RL; manf# RC1206JR-7W0RL -> (none)
- R11, R12: symbol 5uH_LISN-eagle-import:R-EU_R0805 -> Device:R; Manufacturer TE Connectivity / Holsworthy -> (none); Part number (none) -> RT0805BRD07243RL; manf# RQ73C2A243RBTD -> (none)
- R15, R16: symbol 5uH_LISN-eagle-import:R-EU_R0805 -> Device:R; Manufacturer TE -> (none); Part number (none) -> RT0805BRD07274RL; manf# 6-2176091-5 -> (none)
- R17, R18: symbol 5uH_LISN-eagle-import:R-EU_R0805 -> Device:R; Manufacturer TE Connectivity / Holsworthy -> (none); Part number (none) -> AR06DTDV30R1; manf# RQ73C2B30R1BTD -> (none)
- R19, R20, R21, R22, R23, R24, R25, R26: symbol 5uH_LISN-eagle-import:R-EU_R0805 -> Device:R; Manufacturer TE -> (none); Part number (none) -> RT0805BRD07432RL; manf# 8-2176091-3 -> (none)
- R27, R28: symbol 5uH_LISN-eagle-import:R-EU_R0805 -> Device:R; Manufacturer TE Connectivity / Holsworthy -> (none); Part number (none) -> RT1206BRD0718R2L; manf# RQ73C2B18R2BTD -> (none)
- R29, R30: symbol 5uH_LISN-eagle-import:R-EU_R0805 -> Device:R; Manufacturer TE -> (none); Part number (none) -> RT0805BRD07562RL; manf# 9-2176091-4 -> (none)
- R3, R4: symbol 5uH_LISN-rescue:R-Device -> Device:R; Manufacturer KOA -> (none); Part number (none) -> RC1218FK-071RL; manf# WK73S2JTTE1R00F -> (none)
- R31, R32: symbol 5uH_LISN-eagle-import:R-EU_R0805 -> Device:R; Manufacturer TE Connectivity / Holsworthy -> (none); Part number (none) -> RT0805BRE07619RL; manf# RQ73C2A619RBTD -> (none)
- R5, R6: symbol 5uH_LISN-eagle-import:R-EU_R0805 -> Device:R; Manufacturer Panasonic -> (none); Part number (none) -> RT0805BRD07825RL; manf# ERJ-PB6B8250V -> (none)
- R7, R8: symbol 5uH_LISN-eagle-import:R-EU_R0805 -> Device:R; Manufacturer TE Connectivity / Holsworthy -> (none); Part number (none) -> RT1206BRD0712R1L; manf# RQ73C2B12R1BTD -> (none)
Connections:
- net GND: now also J3.1 (P), J8.1 (P), L7.2, L8.2, U1.1, U2.1
- net at C11.1, L11.2: now also J6.1 (P)
- net at C1.1, C3.1, C5.1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: now also J5.1 (P)
- net at C7.2, C9.1: now also L7.1
- net at C11.2, R27.2, R29.2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: now also U1.2
- net at C10.1, C8.2: now also L8.1
- net at C12.2, R28.2, R30.2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: now also U2.2
- net at C2.1, C4.1, C6.1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: now also J4.1 (P)
- net at C12.1, L12.2: now also J7.1 (P)
Other:
- note added: "Banana socket; 4mm; uninsulated; through type; screwed; 16,5mm; nickel plated brass;"
- note removed: "100V or more (250V)"
- note removed: "Banana jacks for soldering: Keystone 575-4 => too short Keystone 575-8"
- note removed: "Hammond case 1590B"
- note removed: "Inductor: Coilcraft 1008PS-105KL"
- note removed: "Mount 1x 100nF = 5uH LISN"
- note removed: "Mount 22uF and 1 Ohm = 5uH LISN"
- note removed: "Mount 2x 0 Ohm and 2x 2.2uF = 5uH LISN"
- note removed: "SMA connector: Würth 60312002114503 TE Connectivity 5-1814832-2 (>2x Cheaper vs Würth 60312002114503)"
- note removed: "TDK NL45323T-102J-PF"
- note removed: "TODO modifications/improvements of 5uH Dual DC-LISN: 1) Add the Simulation in the GitHub repository and check everything (to be checked in EEVBLOG forum) 2) Replace some 1N4148W by BAV99W => Done 3) electronic_eel => Replace Keystone 575-4 with something better ? 3-1) At least allow to have 19.06mm space between Supply+/- 4mm BANANA JACK for BNC adapter... => Done 4) electronic_eel => 4mm input c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"
- note removed: "Würth WE-HCI 744314110 = 5uH LISN"
- company: F.Siebel / B.VERNOUX -> (none)
- moved on the sheet: C1, C2, C3, C4, C5, C6, J1, J2, L1, L10, L11, L12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
